Commit message: camera added

File: ROS1/catkin_ws/src/ackermann_vehicle/ackermann_vehicle_description/urdf/em_3905.urdf.xacro (robot description, xacro)
@@ -327,4 +327,51 @@
 <!--
   <link name="camera_link">
+    <inertial>
+      <mass value="1" />
+       <origin xyz="0 0 0" rpy="0 0 ${pi}"/>
+      <inertia ixx="1" ixy="0" ixz="0" iyy="1" iyz="0" izz="1" />
+    </inertial>
+    <collision>
+      <origin xyz="0 0 0" rpy="0 0 0"/>
+      <geometry>
+        <box size="1 1 1"/>
+      </geometry>
+    </collision>
+    <visual name="my_visual">
+      <origin xyz="0 0 0" rpy="0 0 0"/>
+      <geometry>
+        <box size="0.05 0.05 0.05"/>
+      </geometry>
+    </visual>
+  </link>
+  <joint name="camera_joint" type="fixed">
+    <parent link="chassis"/>
+    <child link= "camera_link" />
+  </joint>
+  <gazebo reference="camera_link">
+    <material>Gazebo/Yellow</material>
+    <sensor type="camera" name="my_camera">
+      <update_rate>10.0</update_rate>
+      <visualize>
+						true
+      </visualize>
+      <plugin name="camera_controller" filename="libgazebo_ros_camera.so">
+        <alwaysOn>true</alwaysOn>
+        <updateRate>0.0</updateRate>
+        <cameraName>vehicle_camera</cameraName>
+        <imageTopicName>image_raw</imageTopicName>
+        <cameraInfoTopicName>camera_info</cameraInfoTopicName>
+        <frameName>camera_link</frameName>
+        <hackBaseline>0.07</hackBaseline>
+        <distortionK1>0.0</distortionK1>
+        <distortionK2>0.0</distortionK2>
+        <distortionK3>0.0</distortionK3>
+        <distortionT1>0.0</distortionT1>
+        <distortionT2>0.0</distortionT2>
+      </plugin>
+    </sensor>
+  </gazebo> -->
+  <!--
+  <link name="camera_link">
     <pose frame="">
 					1 0 0.5 0 -0 0

Commit message: ackerman vehicle works

File: ROS1/catkin_ws/src/ackermann_vehicle/ackermann_vehicle_description/urdf/em_3905.urdf.xacro (robot description, xacro)
@@ -34,7 +34,7 @@
   <!-- chassis_length is measured along the x axis, chassis_width
        along the y axis, and chassis_height along the z axis. -->
-  <xacro:property name="chassis_length" value="1.032"/>
-  <xacro:property name="chassis_width" value="0.672"/>
-  <xacro:property name="chassis_height" value="0.04"/>
+  <xacro:property name="chassis_length" value="0.774"/>
+  <xacro:property name="chassis_width" value="0.504"/>
+  <xacro:property name="chassis_height" value="0.03"/>
   <xacro:property name="chassis_mass" value="2.788"/>
   <!-- battery_dist is the distance between the inner edges of the
@@ -42,12 +42,12 @@
        battery_length is measured along the x axis, battery_width
        along the y axis, and battery_height along the z axis. -->
-  <xacro:property name="battery_x_offset" value="0.22"/>
-  <xacro:property name="battery_dist" value="0.26"/>
-  <xacro:property name="battery_comp_depth" value="0.08"/>
-  <xacro:property name="battery_comp_angle" value="1.3962635"/>
-  <xacro:property name="battery_length" value="0.64"/>
-  <xacro:property name="battery_width" value="0.188"/>
-  <xacro:property name="battery_height" value="0.096"/>
-  <xacro:property name="battery_mass" value="2.01"/>
+  <xacro:property name="battery_x_offset" value="0.165"/>
+  <xacro:property name="battery_dist" value="0.195"/>
+  <xacro:property name="battery_comp_depth" value="0.06"/>
+  <xacro:property name="battery_comp_angle" value="1.04719755"/>
+  <xacro:property name="battery_length" value="0.48"/>
+  <xacro:property name="battery_width" value="0.141"/>
+  <xacro:property name="battery_height" value="0.072"/>
+  <xacro:property name="battery_mass" value="1.5075"/>
   <!-- hub_dia and tire_dia are the diameters of the hub and tire,
        respectively. hex_hub_depth is the distance that the hex hub is
@@ -55,24 +55,24 @@
        is a "zero offset" wheel. hex_hub_depth = tire_width / 2 -
        axle_length. -->
-  <xacro:property name="hub_dia" value="0.38608"/>
-  <xacro:property name="tire_dia" value="0.5842"/>
-  <xacro:property name="tire_width" value="0.3556"/>
-  <xacro:property name="hex_hub_depth" value="0.0578"/>
-  <xacro:property name="wheel_mass" value="1.16"/>
+  <xacro:property name="hub_dia" value="0.28956"/>
+  <xacro:property name="tire_dia" value="0.43815"/>
+  <xacro:property name="tire_width" value="0.2667"/>
+  <xacro:property name="hex_hub_depth" value="0.04335"/>
+  <xacro:property name="wheel_mass" value="0.87"/>
   <!-- hex_hub_dist is the distance between left and right hex hubs when
        the shock absorbers are fully extended. axle_length is the distance
        from a U joint to the corresponding hex hub. wheel_travel is the
        vertical wheel travel. -->
-  <xacro:property name="wheelbase" value="1.34"/>
-  <xacro:property name="hex_hub_dist" value="1.46"/>
-  <xacro:property name="axle_length" value="0.12"/>
-  <xacro:property name="wheel_travel" value="0.336"/>
-  <xacro:property name="shock_z_offset" value="0.262"/>
+  <xacro:property name="wheelbase" value="1.005"/>
+  <xacro:property name="hex_hub_dist" value="1.095"/>
+  <xacro:property name="axle_length" value="0.09"/>
+  <xacro:property name="wheel_travel" value="0.252"/>
+  <xacro:property name="shock_z_offset" value="0.1965"/>
   <!-- shock_eff_limit is 2 * ((shock_stroke / 2) * shock_spring_constant) N.
        shock_stroke is 0.028575 meters. shock_spring_constant, an approximation
        of a Traxxas Ultra Shock shock absorber spring's constant, is
        437.817 N/m. -->
-  <xacro:property name="shock_eff_limit" value="50.0424"/>
-  <xacro:property name="shock_vel_limit" value="4000"/>
+  <xacro:property name="shock_eff_limit" value="37.5318"/>
+  <xacro:property name="shock_vel_limit" value="3000"/>
   <!-- The specifications for a Titan(R) 550 motor could not be found, so the
        stall torque of a Mabuchi Motor(R) RS-550VC-7525 motor was used instead.
@@ -87,6 +87,6 @@
        axle_vel_limit = (2 * pi) * (max_speed / (pi * tire_dia)) =
          244.8696 rad/s -->
-  <xacro:property name="axle_eff_limit" value="20.51064"/>
-  <xacro:property name="axle_vel_limit" value="979.4784"/>
+  <xacro:property name="axle_eff_limit" value="15.38298"/>
+  <xacro:property name="axle_vel_limit" value="734.6088"/>
   <!-- These constants are used to simulate a Traxxas 2056 servo operated at
        6 V. servo_stall_torque is measured in N m. servo_no_load_speed is
@@ -325,102 +325,35 @@
   <xacro:rear_wheel lr_prefix="left" fr_prefix="rear" lr_reflect="1" fr_reflect="-1"/>
   <xacro:rear_wheel lr_prefix="right" fr_prefix="rear" lr_reflect="-1" fr_reflect="-1"/>
-<!--
+  <gazebo>
+    <plugin name="gazebo_ros_control" filename="libgazebo_ros_control.so"/>
+  </gazebo>
+  <joint name="camera_joint" type="fixed">
+    <origin xyz="0.7 0 0.5" rpy="0 0 0"/>
+    <parent link="chassis"/>
+    <child link="camera_link"/>
+  </joint>
   <link name="camera_link">
-    <inertial>
-      <mass value="1" />
-       <origin xyz="0 0 0" rpy="0 0 ${pi}"/>
-      <inertia ixx="1" ixy="0" ixz="0" iyy="1" iyz="0" izz="1" />
-    </inertial>
     <collision>
       <origin xyz="0 0 0" rpy="0 0 0"/>
       <geometry>
-        <box size="1 1 1"/>
+        <box size=".05 .05 .05"/>
       </geometry>
     </collision>
-    <visual name="my_visual">
+    <visual>
       <origin xyz="0 0 0" rpy="0 0 0"/>
       <geometry>
-        <box size="0.05 0.05 0.05"/>
+        <box size=".05 .05 .05"/>
       </geometry>
+      <material name="blue"/>
     </visual>
+    <inertial>
+      <mass value="0.05" />
+      <origin xyz="0 0 0" rpy="0 0 0"/>
+      <inertia ixx="0.001" ixy="0" ixz="0" iyy="0.001" iyz="0" izz="0.001"/>
+      <box_inertia x=".05" y=".05" z=".05" m="0.05" />
+    </inertial>
   </link>
-  <joint name="camera_joint" type="fixed">
-    <parent link="chassis"/>
-    <child link= "camera_link" />
-  </joint>
   <gazebo reference="camera_link">
-    <material>Gazebo/Yellow</material>
-    <sensor type="camera" name="my_camera">
-      <update_rate>10.0</update_rate>
-      <visualize>
-						true
-      </visualize>
-      <plugin name="camera_controller" filename="libgazebo_ros_camera.so">
-        <alwaysOn>true</alwaysOn>
-        <updateRate>0.0</updateRate>
-        <cameraName>vehicle_camera</cameraName>
-        <imageTopicName>image_raw</imageTopicName>
-        <cameraInfoTopicName>camera_info</cameraInfoTopicName>
-        <frameName>camera_link</frameName>
-        <hackBaseline>0.07</hackBaseline>
-        <distortionK1>0.0</distortionK1>
-        <distortionK2>0.0</distortionK2>
-        <distortionK3>0.0</distortionK3>
-        <distortionT1>0.0</distortionT1>
-        <distortionT2>0.0</distortionT2>
-      </plugin>
-    </sensor>
-  </gazebo> -->
-  <!--
-  <link name="camera_link">
-    <pose frame="">
-					1 0 0.5 0 -0 0
-    </pose>
-    <inertial>
-      <inertia>
-        <ixx>
-							1
-        </ixx>
-        <ixy>
-							0
-        </ixy>
-        <ixz>
-							0
-        </ixz>
-        <iyy>
-							1
-        </iyy>
-        <iyz>
-							0
-        </iyz>
-        <izz>
-							1
-        </izz>
-      </inertia>
-      <mass>
-						1.0
-      </mass>
-    </inertial>
-    <collision name="my_collision">
-      <pose>
-						0 0 0.5 0 0 0
-      </pose>
-      <geometry>
-        <box>
-          <size>
-								1 1 1
-          </size>
-        </box>
-      </geometry>
-    </collision>
-    <visual name="my_visual">
-      <geometry>
-        <box>
-          <size>
-								0.005 0.005 0.005
-          </size>
-        </box>
-      </geometry>
-    </visual>
+    <material>Gazebo/Red</material>
     <sensor type="camera" name="my_camera">
       <camera>
@@ -445,56 +378,25 @@
         </clip>
       </camera>
-      <always_on>
-						1
-      </always_on>
-      <update_rate>
-						10
-      </update_rate>
+      <update_rate>10.0</update_rate>
+      <always_on>1</always_on>
       <visualize>
-						true
+           true
       </visualize>
+      <plugin name="camera_controller" filename="libgazebo_ros_camera.so">
+        <alwaysOn>true</alwaysOn>
+        <updateRate>0.0</updateRate>
+        <visualize>true</visualize>
+        <cameraName>vehicle_camera</cameraName>
+        <imageTopicName>image_raw</imageTopicName>
+        <cameraInfoTopicName>camera_info</cameraInfoTopicName>
+        <frameName>camera_link</frameName>
+        <hackBaseline>0.07</hackBaseline>
+        <distortionK1>0.0</distortionK1>
+        <distortionK2>0.0</distortionK2>
+        <distortionK3>0.0</distortionK3>
+        <distortionT1>0.0</distortionT1>
+        <distortionT2>0.0</distortionT2>
+      </plugin>
     </sensor>
-  </link>
-  <gazebo>
-    <plugin name="camera_controller" filename="libgazebo_ros_camera.so">
-      <alwaysOn>
-							true
-      </alwaysOn>
-      <updateRate>
-							0.0
-      </updateRate>
-      <cameraName link= "vehicle_camera" />
-      <imageTopicName link= "image_raw" />
-      <cameraInfoTopicName link= "camera_info" />
-      <frameName link= "camera_link" />
-      <hackBaseline>
-							0.07
-      </hackBaseline>
-      <distortionK1>
-							0.0
-      </distortionK1>
-      <distortionK2>
-							0.0
-      </distortionK2>
-      <distortionK3>
-							0.0
-      </distortionK3>
-      <distortionT1>
-							0.0
-      </distortionT1>
-      <distortionT2>
-							0.0
-      </distortionT2>
-    </plugin>
-  </gazebo> -->
-  <!-- <gazebo reference="camera_link">
-    <material>Gazebo/White</material>
-  </gazebo>
-  <joint name="camera_joint" type="fixed">
-    <parent link="chassis"/>
-    <child link= "camera_link" />
-  </joint> -->
-  <gazebo>
-    <plugin name="gazebo_ros_control" filename="libgazebo_ros_control.so"/>
   </gazebo>
 </robot>
